File: SENSOR CONNECTOR/con connector.brd (EAGLE design)
At the start: 77.5 x 69.1 mm, 31 parts, among them IC1 7805TV, IC2 7805TV, IC3 7805TV, T1 BC547, T2 BC547, T3 BC547

Commit message: 24/10/19/11:25
Parts:
- removed C1: 100uF, rcl:E2,5-7
- removed C4: 10uF, rcl:E2,5-6
- removed D1: 1N4733A, diode:DO41Z10
- removed IC1: 7805TV, linear:TO220V
- removed JP1, JP2, JP7: (no value), pinhead:1X02
- removed R1: 10k, rcl:0207/12
- removed T1: BC547, transistor:TO92
- removed U$1: DC-DC-STEP-DOWN-LM2596, diy-modules:DC-DC-STEP-DOWN-LM2596
- moved D2 1.73 mm to (63.9, 30.5)
- moved IC2 1.73 mm to (75.2, 30.8)
- moved C5 1.73 mm to (58.6, 27.4)
- moved JP4 1.73 mm to (6.04, 25.2)
- moved R2 1.73 mm to (68.0, 30.3)
- moved C2 1.73 mm to (57.4, 35.2), turned to 270 degrees
- moved JP8 1.73 mm to (57.5, 41.9)
- moved T2 1.73 mm to (63.9, 41.9)
- moved U$2 1.73 mm to (31.3, 32.9)
- moved JP3 1.73 mm to (6.10, 40.6)
- turned C3 to 270 degrees
Connections:
- removed net N$1: C1.+, IC1.1, U$1.OUT+
- removed net N$15: R1.2, T1.2
- removed net N$19: JP1.1, JP1.2, U$1.IN+
- removed net N$2: C1.-, C4.-, D1.A, IC1.2, U$1.OUT-
- removed net N$21: JP2.1, JP2.2, U$1.IN-
- removed net N$26: JP7.1, JP7.2, T1.3
- removed net N$4: C2.-, C5.-, D2.A, IC2.2, U$2.OUT-
- removed net N$6: C3.-, C6.-, D3.A, IC3.2, U$3.OUT-
- removed net N$7: C4.+, D1.C, IC1.3, R1.1
- new net GND: C2.-, C3.-, C5.-, C6.-, D2.A, D3.A, IC2.2, IC3.2, U$2.OUT-, U$3.OUT-
- net N$18: no longer T1.1
Routing:
- net GND: track 0.00 -> 69.6 mm
- net N$1: track 41.2 -> 0.00 mm
- net N$2: track 38.0 -> 0.00 mm
- net N$6: track 37.6 -> 0.00 mm
- net N$4: track 37.3 -> 0.00 mm
- net N$18: track 75.3 -> 43.2 mm
- net N$7: track 17.0 -> 0.00 mm
- net N$5: track 40.0 -> 27.5 mm
- net N$3: track 39.6 -> 27.3 mm
- net N$21: track 8.08 -> 0.00 mm
- net N$19: track 8.07 -> 0.00 mm
- net N$15: track 6.42 -> 0.00 mm
- net N$26: track 6.32 -> 0.00 mm
- added copper zone on layer 16, net GND
- removed copper zone on layer 16, net N$10
Other:
- board size 77.5 x 69.1 mm -> 77.5 x 49.1 mm
