File: MAIN CONTROLLER/fms controller.brd (EAGLE design)
At the start: 145.3 x 80.3 mm, 54 parts, among them IC3 7805TV, IC5 7805TV, Q1 16MHz, T1 BC547, T2 BC547, T3 BC547, T4 BC547, T5 BC547, T6 BC547, T7 BC547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

Commit message: 27/11/19/10:07
Parts:
- added C4, C5: 10uF, rcl:E2-5
- added TP1, TP2, TP3: TPPAD1-13, testpad:P1-13
- added TP5: TPPAD1-20, testpad:P1-20
- moved JP7 4.31 mm to (86.3, 78.1)
- moved JP6 2.11 mm to (82.1, 75.8)
Connections:
- new net N$18: C5.+, TP2.TP, TP5.TP, U$1.J2.3
- net GND: now also C4.-, C5.-, TP3.TP
- net VCC: now also C4.+, TP1.TP; no longer U$1.J2.3
Routing:
- net N$18: track 0.00 -> 29.1 mm
- net VCC: track 303.4 -> 284.7 mm
- net RST: track 9.53 -> 8.51 mm
- net SDA: track 36.9 -> 36.3 mm
