File: MAIN CONTROLLER/fms controller.sch (EAGLE design)
At the start: 60 parts, among them IC3 7805TV, IC5 7805TV, Q1 16MHz, T1 BC547, T2 BC547, T3 BC547, T4 BC547, T5 BC547, T6 BC547, T7 BC547, U1 328P

Commit message: 04/01/2020/08:38
Parts:
- removed JP13: (no value), pinhead:PINHD-1X2
- removed JP2: START, pinhead:PINHD-1X4
- removed T7: BC547, transistor:BC547
- removed TP1, TP2, TP3: TPPAD1-13, testpad:TPPAD1-13
- removed TP5: TPPAD1-20, testpad:TPPAD1-20
- added C10, C11, C17, C21, C6, C7, C8, C9: 100nF, rcl:C-EU025-040X050
- added C16, C18, C19, C20: 22pF, capacitor-wima:C2,5-3
- added C22: 10uF, rcl:CPOL-USE2-5
- added DZ1, DZ4, DZ5: 5.1, diode:ZPD
- added IC1, IC2: LM2936MP-3.3, national-semiconductor:LM2936MP-3.3
- added JP16: (no value), pinhead:PINHD-2X3
- added JP17: (no value), pinhead:PINHD-2X2
- added LED3, LED4, LED5, LED6: (no value), led:LED3MM
- added Q2, Q3: 12MHz, special:XTAL/S
- added R14, R16, R18: 100K, rcl:R-EU_0309/10
- added R15, R17, R4: 1M, rcl:R-EU_0309/10
- added R19, R20, R21, R22, R23: 1k, rcl:R-EU_0309/10
- added T8: BC547, transistor:BC547
- added U$2, U$3: CH340G, ch340g:CH340G
- C4: value 10uF -> 100uF
- JP1: value STOP -> (none); device pinhead:PINHD-1X4 -> pinhead:PINHD-1X2
- JP10, JP12, JP9: device pinhead:PINHD-1X2 -> pinhead:PINHD-1X4
Connections:
- removed net N$2: R1.2, T7.B
- removed net N$4: CON.IN+, JP1.3, JP1.4
- removed net N$6: CON.IN-, JP1.1, JP1.2
- new net ACCIN: JP16.1, JP16.2, R4.1
- new net ACCOUT: C8.1, DZ1.C, R14.1, R4.2, U1.PC1(ADC1)
- new net ALTIN: JP16.3, JP16.4, R17.1
- new net ALTOUT: C9.1, DZ4.C, R17.2, R18.1, U1.PC2(ADC2)
- new net D+MAIN: JP12.3, U$2.D+
- new net D+RF: JP9.2, U$3.D+
- new net D-MAIN: JP12.2, U$2.D-
- new net D-RF: JP9.3, U$3.D-
- new net DUMPIN: JP16.5, JP16.6, R15.1
- new net DUMPOUT: C10.1, DZ5.C, R15.2, R16.1, U1.PC3(ADC3)
- new net N$19: C7.1, U1.AREF
- new net N$20: C19.2, Q3.2, U$3.XI
- new net N$22: C20.2, Q3.1, U$3.XO
- new net N$23: C16.2, Q2.2, U$2.XI
- new net N$28: C18.2, Q2.1, U$2.XO
- new net N$31: C21.1, U$2.DTR
- new net N$33: C22.-, T8.C
- new net N$37: LED4.A, R20.1
- new net N$39: LED3.A, R19.1
- new net N$42: LED5.A, R21.1
- new net N$43: LED6.A, R22.1
- new net N$44: R23.1, T8.B
- new net RXRF: JP10.3, LED5.C, U$3.TX
- new net TXRF: JP10.2, LED6.C, U$3.RX
- new net VSS: C17.1, IC2.GND@1, IC2.GND@2, U$2.V3, U$3.V3
- net ACCEXT: no longer JP9.1, JP9.2
- net ALTEXT: no longer JP10.1, JP10.2
- net DUMPEXT: now also R23.2; no longer JP11.1, JP11.2
- net GND: now also C10.2, C11.2, C16.1, C17.2, C18.1, C19.1, C20.1, C6.2, C7.2, C8.2, C9.2, CON.IN-, DZ1.A, DZ4.A, DZ5.A, IC1.VIN, IC2.VIN, JP10.1, JP17.1, JP17.2, JP17.3, JP17.4, JP9.1, LATTEPANDA1.IN-, R14.2, R16.2, R18.2, T8.E, U$2.GND, U$3.GND; no longer JP12.2, T7.E, TP3.TP
- net LOAD: now also R1.2; no longer T7.C
- net N$1: now also JP11.1, JP11.2, LATTEPANDA1.IN+; no longer JP2.1, JP2.2, LATTEPANDA1.IN-
- net N$18: now also IC1.GND@1, IC1.GND@2; no longer TP2.TP, TP5.TP
- net N$3: now also CON.IN+, JP1.1, JP1.2; no longer JP2.3, JP2.4, LATTEPANDA1.IN+
- net RSTEXT: now also C21.2, C22.+
- net RXDEXT: now also LED3.C, U$2.TX; no longer JP13.1
- net TXDEXT: now also LED4.C, U$2.RX; no longer JP13.2
- net VCC: now also C11.1, C6.1, IC1.VO, IC2.VO, JP10.4, R19.2, R20.2, R21.2, R22.2, U$2.VCC, U$3.VCC; no longer JP5.3, JP5.5, JP5.7, TP1.TP
Other:
- note added: "Controller"
- note added: "Port & Jumper"
- note added: "Power & Loading Mechanism"
- note added: "Real Time Clock"
- note added: "Sensor Sensing"
- note added: "USB TTL"
- moved on the sheet: C1, C12, C13, C14, C15, C2, C3, C4, C5, CON, D1, DZ2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
