File: RF LINK/rf exca/rf exca.brd (EAGLE design)
At the start: 117.4 x 67.9 mm, 33 parts, among them IC1 7805T, IC2 7805T, Q1 16MHz, T1 BC547, U1 328P

Commit message: 06/12/19/14:04
Parts:
- removed D4: 5KP36A, diode:P6T15
- removed JP10: RES10kRST, pinhead:1X02
- removed JP11: RSTEXT, pinhead:1X02
- removed T1: BC547, transistor:TO92
- added JP1: HORN, pinhead:1X04
- added R4, R5, R6: 10k, rcl:0207/12
- JP2: value HORN -> VS
- JP3: value VS -> RST; device pinhead:1X04 -> pinhead:1X02
- JP8: value (none) -> 10K; device pinhead:2X05 -> pinhead:1X02
- JP9: value (none) -> LCDI2C; device pinhead:2X05 -> pinhead:1X02
- moved IC2 100.6 mm to (27.4, -5.75), turned to 180 degrees
- moved JP3 72.6 mm to (76.6, 52.1), turned to 0 degrees
- moved C4 67.4 mm to (12.9, 5.75), turned to 180 degrees
- moved JP7 67.3 mm to (62.8, 2.60), turned to 180 degrees
- moved C6 63.5 mm to (56.4, 2.47), turned to 1.7 degrees
- moved R2 63.5 mm to (28.2, 10.2)
- moved LED1 63.4 mm to (39.2, 10.3)
- moved JP4 52.6 mm to (61.0, 30.7), turned to 180 degrees
- moved D2 51.1 mm to (62.7, 6.99), turned to 359.9 degrees
- moved JP2 43.9 mm to (13.2, 60.7), turned to 0 degrees
- moved JP13 35.9 mm to (76.5, 56.6), turned to 0 degrees
- moved R3 34.4 mm to (66.8, 20.9), turned to 270 degrees
- moved JP12 31.3 mm to (76.6, 46.8), turned to 270 degrees
- moved IC1 30.3 mm to (40.6, -5.67)
- moved U$2 28.4 mm to (12.8, 35.4), turned to 270 degrees
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Connections:
- removed net GP: JP10.1, JP9.10, JP9.4, JP9.6, JP9.8, JP9.9
- removed net N$13: R1.2, T1.2
- removed net N$3: JP2.3, JP2.4, U$1.IN+
- removed net PD2: JP8.1, U1.4
- removed net PD3: JP8.2, U1.5
- removed net PD4: T1.3, U1.6
- removed net RSTMCU: JP10.2, JP11.2, JP9.7
- removed net RX: JP8.5, U1.2
- removed net RX1: JP4.3, JP9.1
- removed net TX: JP8.3, U1.3
- removed net TX1: JP4.2, JP9.2
- new net ADC(HORN): R5.1, R6.2, U1.26
- new net HORN(IN+): JP1.3, JP1.4, R5.2, U$1.IN+
- new net PD5: R1.2, R4.2, U1.11
- new net RXGPS: JP4.2, U1.5
- new net SCL: JP9.1, U1.28
- new net SDA: JP9.2, U1.27
- new net TXGPS: JP4.3, U1.4
- net GND: now also JP3.1, R4.1, R6.1; no longer JP11.1, T1.1
- net N$4: now also JP1.1, JP1.2; no longer JP2.1, JP2.2
- net N$5: now also JP2.3, JP2.4; no longer D4.C, JP3.3, JP3.4
- net N$6: now also JP2.1, JP2.2; no longer D4.A, JP3.1, JP3.2
- net RST: now also JP3.2, JP8.1; no longer JP8.7
- net UARTRX: now also U1.2; no longer JP9.5
- net UARTTX: now also U1.3; no longer JP9.3
- net VCC: now also JP8.2; no longer JP8.10, JP8.4, JP8.6, JP8.8, JP8.9
Routing:
- net GND: track 182.4 -> 9.98 mm
- net VCC: track 250.7 -> 135.6 mm
- net PD4: track 91.4 -> 0.00 mm
- net ADC(HORN): track 0.00 -> 86.3 mm
- net TX1: track 49.8 -> 0.00 mm
- net RX1: track 49.4 -> 0.00 mm
- net PD5: track 0.00 -> 43.9 mm
- net HORN(IN+): track 0.00 -> 42.4 mm
- net N$10: track 46.6 -> 15.2 mm
- net TXGPS: track 0.00 -> 27.4 mm
- net N$11: track 23.4 -> 48.1 mm
- net RXGPS: track 0.00 -> 24.2 mm
- net PD3: track 22.4 -> 0.00 mm
- net N$15: track 48.2 -> 26.3 mm
- net N$3: track 20.1 -> 0.00 mm
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Other:
- board size 117.4 x 67.9 mm -> 117.4 x 67.5 mm

Commit message: 04/01/2020/08:38
Parts:
- R5: value 10k -> 1M
- R6: value 10k -> 100K
- moved C2 5.72 mm to (75.8, 19.7), turned to 0 degrees
- moved C1 1.93 mm to (71.2, 26.2)
- moved JP4 0.75 mm to (61.0, 31.4)
Connections:
- net RXGPS: now also JP4.3; no longer JP4.2
- net TXGPS: now also JP4.2; no longer JP4.3
Routing:
- net TXGPS: track 27.4 -> 24.5 mm
- net RXGPS: track 24.2 -> 26.2 mm, vias 0 -> 2
- net N$1: track 10.2 -> 11.4 mm
Changed lines of the file:
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@@
 <drawing>
 <settings>
-<setting alwaysvectorfont="yes"/>
+<setting alwaysvectorfont="no"/>
 <setting verticaltext="up"/>
 </settings>
@@
 </autorouter>
 <elements>
-<element name="C1" library="rcl" library_urn="urn:adsk.eagle:library:334" package="C025-024X044" package3d_urn="urn:adsk.eagle:package:23630/1" value="22pF" x="71.3130375" y="28.160975" rot="R90">
-<attribute name="SPICEPREFIX" value="C" x="71.3130375" y="28.160975" size="1.778" layer="27" rot="R90" display="off"/>
-</element>
-<element name="C2" library="rcl" library_urn="urn:adsk.eagle:library:334" package="C025-024X044" package3d_urn="urn:adsk.eagle:package:23630/1" value="22pF" x="71.26731875" y="23.215590625" rot="R270">
-<attribute name="SPICEPREFIX" value="C" x="71.26731875" y="23.215590625" size="1.778" layer="27" rot="R270" display="off"/>
+<element name="C1" library="rcl" library_urn="urn:adsk.eagle:library:334" package="C025-024X044" package3d_urn="urn:adsk.eagle:package:23630/1" value="22pF" x="71.20635625" y="26.230575" rot="R90">
+<attribute name="SPICEPREFIX" value="C" x="71.20635625" y="26.230575" size="1.778" layer="27" rot="R90" display="off"/>
+</element>
+<element name="C2" library="rcl" library_urn="urn:adsk.eagle:library:334" package="C025-024X044" package3d_urn="urn:adsk.eagle:package:23630/1" value="22pF" x="75.76311875" y="19.679909375">
+<attribute name="SPICEPREFIX" value="C" x="75.76311875" y="19.679909375" size="1.778" layer="27" display="off"/>
 </element>
 <element name="C4" library="rcl" library_urn="urn:adsk.eagle:library:334" package="E5-13" package3d_urn="urn:adsk.eagle:package:23375/1" value="2200uF" x="12.915896875" y="5.750559375" rot="R180">
@@
 <element name="D1" library="diode" library_urn="urn:adsk.eagle:library:210" package="DO41Z10" package3d_urn="urn:adsk.eagle:package:43341/1" value="1N4733A" x="59.687465625" y="19.626575" rot="R90"/>
 <element name="D2" library="diode" library_urn="urn:adsk.eagle:library:210" package="DO41Z10" package3d_urn="urn:adsk.eagle:package:43341/1" value="1N4733A" x="62.69736875" y="6.98501875" rot="R359.9"/>
-<element name="JP4" library="pinhead" library_urn="urn:adsk.eagle:library:325" package="1X04" package3d_urn="urn:adsk.eagle:package:22407/2" value="GPS" x="60.970159375" y="30.69845" rot="R180"/>
+<element name="JP4" library="pinhead" library_urn="urn:adsk.eagle:library:325" package="1X04" package3d_urn="urn:adsk.eagle:package:22407/2" value="GPS" x="60.970159375" y="31.44775" rot="R180"/>
 <element name="JP5" library="pinhead" library_urn="urn:adsk.eagle:library:325" package="1X06" package3d_urn="urn:adsk.eagle:package:22472/2" value="NRF24L01" x="103.1519375" y="43.428915625" rot="R180"/>
 <element name="JP6" library="pinhead" library_urn="urn:adsk.eagle:library:325" package="1X02" package3d_urn="urn:adsk.eagle:package:22435/2" value="PWR NRF" x="96.753671875" y="55.227215625" rot="R90"/>
@@
 <attribute name="SPICEPREFIX" value="R" x="63.3069625" y="20.939759375" size="1.778" layer="27" rot="R90" display="off"/>
 </element>
-<element name="R5" library="rcl" library_urn="urn:adsk.eagle:library:334" package="0207/12" package3d_urn="urn:adsk.eagle:package:23489/1" value="10k" x="49.55031875" y="20.792440625" rot="R90">
+<element name="R5" library="rcl" library_urn="urn:adsk.eagle:library:334" package="0207/12" package3d_urn="urn:adsk.eagle:package:23489/1" value="1M" x="49.55031875" y="20.792440625" rot="R90">
 <attribute name="SPICEPREFIX" value="R" x="49.55031875" y="20.792440625" size="1.778" layer="27" rot="R90" display="off"/>
 </element>
-<element name="R6" library="rcl" library_urn="urn:adsk.eagle:library:334" package="0207/12" package3d_urn="urn:adsk.eagle:package:23489/1" value="10k" x="53.00471875" y="20.7899" rot="R90">
+<element name="R6" library="rcl" library_urn="urn:adsk.eagle:library:334" package="0207/12" package3d_urn="urn:adsk.eagle:package:23489/1" value="100K" x="53.00471875" y="20.7899" rot="R90">
 <attribute name="SPICEPREFIX" value="R" x="53.00471875" y="20.7899" size="1.778" layer="27" rot="R90" display="off"/>
 </element>
@@
 <wire x1="81.147921875" y1="30.274259375" x2="76.542896875" y2="30.274259375" width="0.762" layer="16"/>
 <wire x1="76.542896875" y1="30.274259375" x2="75.93330625" y2="29.66466875" width="0.762" layer="16"/>
-<wire x1="71.3130375" y1="29.430975" x2="75.6996125" y2="29.430975" width="0.762" layer="16"/>
 <wire x1="75.6996125" y1="29.430975" x2="75.93330625" y2="29.66466875" width="0.762" layer="16"/>
+<wire x1="71.20635625" y1="27.500575" x2="73.37045" y2="29.66466875" width="0.762" layer="16"/>
+<wire x1="73.37045" y1="29.66466875" x2="75.93330625" y2="29.66466875" width="0.762" layer="16"/>
 </signal>
 <signal name="N$2">
@@
 <wire x1="77.1906" y1="27.71901875" x2="81.13268125" y2="27.71901875" width="0.762" layer="16"/>
 <wire x1="81.13268125" y1="27.71901875" x2="81.147921875" y2="27.734259375" width="0.762" layer="16"/>
-<wire x1="73.294228125" y1="21.945590625" x2="71.26731875" y2="21.945590625" width="0.762" layer="16"/>
-<wire x1="75.93330625" y1="24.58466875" x2="73.294228125" y2="21.945590625" width="0.762" layer="16"/>
+<wire x1="77.03311875" y1="19.679909375" x2="77.03311875" y2="23.48485625" width="0.762" layer="16"/>
+<wire x1="77.03311875" y1="23.48485625" x2="75.93330625" y2="24.58466875" width="0.762" layer="16"/>
 </signal>
 <signal name="N$4">
@@
 <contactref element="JP4" pad="1"/>
 <contactref element="JP13" pad="2"/>
-<wire x1="64.780159375" y1="30.69845" x2="69.43596875" y2="35.354259375" width="0.762" layer="16"/>
-<wire x1="69.43596875" y1="35.354259375" x2="81.147921875" y2="35.354259375" width="0.762" layer="16"/>
 <wire x1="81.147921875" y1="35.354259375" x2="82.8268625" y2="35.354259375" width="0.762" layer="16"/>
 <wire x1="82.8268625" y1="35.354259375" x2="82.85988125" y2="35.321240625" width="0.762" layer="16"/>
@@
 <wire x1="84.94268125" y1="25.58541875" x2="84.94268125" y2="15.9512" width="0.762" layer="16"/>
 <wire x1="84.94268125" y1="15.9512" x2="82.654140625" y2="13.662659375" width="0.762" layer="16"/>
+<wire x1="64.780159375" y1="31.44775" x2="68.68666875" y2="35.354259375" width="0.762" layer="16"/>
+<wire x1="68.68666875" y1="35.354259375" x2="81.147921875" y2="35.354259375" width="0.762" layer="16"/>
 </signal>
 <signal name="MOSI">
@@
 <signal name="TXGPS">
 <contactref element="U1" pad="4"/>
-<contactref element="JP4" pad="3"/>
-<wire x1="59.7027" y1="32.24021875" x2="59.7027" y2="30.700990625" width="0.762" layer="16"/>
-<wire x1="59.7027" y1="30.700990625" x2="59.700159375" y2="30.69845" width="0.762" layer="16"/>
-<wire x1="81.147921875" y1="42.974259375" x2="70.436740625" y2="42.974259375" width="0.762" layer="16"/>
-<wire x1="70.436740625" y1="42.974259375" x2="59.7027" y2="32.24021875" width="0.762" layer="16"/>
+<contactref element="JP4" pad="2"/>
+<wire x1="62.240159375" y1="31.44775" x2="62.240159375" y2="32.771078125" width="0.762" layer="16"/>
+<wire x1="62.240159375" y1="32.771078125" x2="72.443340625" y2="42.974259375" width="0.762" layer="16"/>
+<wire x1="72.443340625" y1="42.974259375" x2="81.147921875" y2="42.974259375" width="0.762" layer="16"/>
 </signal>
 <signal name="RST">
@@
 <signal name="RXGPS">
 <contactref element="U1" pad="5"/>
-<contactref element="JP4" pad="2"/>
-<wire x1="62.240159375" y1="30.69845" x2="62.240159375" y2="31.87191875" width="0.762" layer="16"/>
-<wire x1="62.240159375" y1="30.69845" x2="63.433953125" y2="31.89224375" width="0.762" layer="16"/>
-<wire x1="63.433953125" y1="31.89224375" x2="63.433953125" y2="32.018065625" width="0.762" layer="16"/>
-<wire x1="63.433953125" y1="32.018065625" x2="71.850146875" y2="40.434259375" width="0.762" layer="16"/>
-<wire x1="71.850146875" y1="40.434259375" x2="81.147921875" y2="40.434259375" width="0.762" layer="16"/>
+<contactref element="JP4" pad="3"/>
+<wire x1="59.700159375" y1="31.44775" x2="59.700159375" y2="33.0708" width="0.762" layer="16"/>
+<wire x1="59.700159375" y1="33.0708" x2="66.9036" y2="40.274240625" width="0.762" layer="16"/>
+<via x="66.9036" y="40.274240625" extent="1-16" drill="1" diameter="1.524"/>
+<wire x1="66.9036" y1="40.274240625" x2="73.6473" y2="40.274240625" width="0.762" layer="1"/>
+<wire x1="73.6473" y1="40.274240625" x2="73.75398125" y2="40.167559375" width="0.762" layer="1"/>
+<via x="73.75398125" y="40.167559375" extent="1-16" drill="1" diameter="1.524"/>
+<wire x1="73.75398125" y1="40.167559375" x2="80.881221875" y2="40.167559375" width="0.762" layer="16"/>
+<wire x1="80.881221875" y1="40.167559375" x2="81.147921875" y2="40.434259375" width="0.762" layer="16"/>
 </signal>
 <signal name="UARTTX">
