File: RF LINK/rf exca/rf exca.sch (EAGLE design)
At the start: 33 parts, among them IC1 7805T, IC2 7805T, Q1 16MHz, T1 BC547, U1 328P

Commit message: 06/12/19/14:04
Parts:
- removed D4: 5KP36A, diode:5KPXX
- removed JP10: RES10kRST, pinhead:PINHD-1X2
- removed JP11: RSTEXT, pinhead:PINHD-1X2
- removed T1: BC547, transistor:BC547
- added JP1: HORN, pinhead:PINHD-1X4
- added R4, R5, R6: 10k, rcl:R-EU_0207/12
- JP2: value HORN -> VS
- JP3: value VS -> RST; device pinhead:PINHD-1X4 -> pinhead:PINHD-1X2
- JP8: value (none) -> 10K; device pinhead:PINHD-2X5 -> pinhead:PINHD-1X2
- JP9: value (none) -> LCDI2C; device pinhead:PINHD-2X5 -> pinhead:PINHD-1X2
Connections:
- removed net GP: JP10.1, JP9.10, JP9.4, JP9.6, JP9.8, JP9.9
- removed net N$13: R1.2, T1.B
- removed net N$3: JP2.3, JP2.4, U$1.IN+
- removed net PD2: JP8.1, U1.PD2(INT0)
- removed net PD3: JP8.2, U1.PD3(INT1)
- removed net PD4: T1.C, U1.PD4(XCK/T0)
- removed net RSTMCU: JP10.2, JP11.2, JP9.7
- removed net RX: JP8.5, U1.PD0(RXD)
- removed net RX1: JP4.3, JP9.1
- removed net TX: JP8.3, U1.PD1(TXD)
- removed net TX1: JP4.2, JP9.2
- new net ADC(HORN): R5.1, R6.2, U1.PC3(ADC3)
- new net HORN(IN+): JP1.3, JP1.4, R5.2, U$1.IN+
- new net PD5: R1.2, R4.2, U1.PD5(T1)
- new net RXGPS: JP4.2, U1.PD3(INT1)
- new net SCL: JP9.1, U1.PC5(ADC5/SCL)
- new net SDA: JP9.2, U1.PC4(ADC4/SDA)
- new net TXGPS: JP4.3, U1.PD2(INT0)
- net GND: now also JP3.1, R4.1, R6.1; no longer JP11.1, T1.E
- net N$4: now also JP1.1, JP1.2; no longer JP2.1, JP2.2
- net N$5: now also JP2.3, JP2.4; no longer D4.C, JP3.3, JP3.4
- net N$6: now also JP2.1, JP2.2; no longer D4.A, JP3.1, JP3.2
- net RST: now also JP3.2, JP8.1; no longer JP8.7
- net UARTRX: now also U1.PD0(RXD); no longer JP9.5
- net UARTTX: now also U1.PD1(TXD); no longer JP9.3
- net VCC: now also JP8.2; no longer JP8.10, JP8.4, JP8.6, JP8.8, JP8.9
Other:
- moved on the sheet: JP13, JP2, JP4

Commit message: 04/01/2020/08:38
Parts:
- R5: value 10k -> 1M
- R6: value 10k -> 100K
Connections:
- net RXGPS: now also JP4.3; no longer JP4.2
- net TXGPS: now also JP4.2; no longer JP4.3
Changed lines of the file:
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@@
 <part name="R4" library="rcl" library_urn="urn:adsk.eagle:library:334" deviceset="R-EU_" device="0207/12" package3d_urn="urn:adsk.eagle:package:23489/1" value="10k"/>
 <part name="GND2" library="supply1" library_urn="urn:adsk.eagle:library:371" deviceset="GND" device=""/>
-<part name="R5" library="rcl" library_urn="urn:adsk.eagle:library:334" deviceset="R-EU_" device="0207/12" package3d_urn="urn:adsk.eagle:package:23489/1" value="10k"/>
-<part name="R6" library="rcl" library_urn="urn:adsk.eagle:library:334" deviceset="R-EU_" device="0207/12" package3d_urn="urn:adsk.eagle:package:23489/1" value="10k"/>
+<part name="R5" library="rcl" library_urn="urn:adsk.eagle:library:334" deviceset="R-EU_" device="0207/12" package3d_urn="urn:adsk.eagle:package:23489/1" value="1M"/>
+<part name="R6" library="rcl" library_urn="urn:adsk.eagle:library:334" deviceset="R-EU_" device="0207/12" package3d_urn="urn:adsk.eagle:package:23489/1" value="100K"/>
 <part name="GND3" library="supply1" library_urn="urn:adsk.eagle:library:371" deviceset="GND" device=""/>
 <part name="JP1" library="pinhead" library_urn="urn:adsk.eagle:library:325" deviceset="PINHD-1X4" device="" package3d_urn="urn:adsk.eagle:package:22407/2" value="HORN"/>
@@
 </segment>
 <segment>
-<pinref part="JP4" gate="A" pin="3"/>
-<wire x1="-33.02" y1="25.4" x2="-25.4" y2="25.4" width="0.1524" layer="91"/>
-<label x="-25.4" y="25.4" size="1.778" layer="95" xref="yes"/>
+<pinref part="JP4" gate="A" pin="2"/>
+<wire x1="-33.02" y1="22.86" x2="-25.4" y2="22.86" width="0.1524" layer="91"/>
+<label x="-25.4" y="22.86" size="1.778" layer="95" xref="yes"/>
 </segment>
 </net>
@@
 </segment>
 <segment>
-<pinref part="JP4" gate="A" pin="2"/>
-<wire x1="-33.02" y1="22.86" x2="-25.4" y2="22.86" width="0.1524" layer="91"/>
-<label x="-25.4" y="22.86" size="1.778" layer="95" xref="yes"/>
-</segment>
-</net>
+<pinref part="JP4" gate="A" pin="3"/>
+<wire x1="-33.02" y1="25.4" x2="-25.4" y2="25.4" width="0.1524" layer="91"/>
+<label x="-25.4" y="25.4" size="1.778" layer="95" xref="yes"/>
+</segment>
+</net>
